File: 24_wires_away.kicad_pcb (KiCad board)
At the start: 2 copper layers, 29.2 x 57.2 mm, 4 parts, among them J1 Conn_01x24_Pin, U1 Elite-C, U3 74HCT138, U4 74HCT138

Commit message: more changes
Parts:
- added J3: Conn_01x06_Pin, Library:SolderWire-SMD-0.127sqmm_1x06_P3.7mm_D0.48mm_OD1mm, F.Cu at (138.6, 58.6)
- added U2: TXS0108EPW, Package_SO:TSSOP-20_4.4x6.5mm_P0.65mm, F.Cu at (135.3, 96.0)
- U1: footprint Keebio:Elite-C-castellated-24pin -> Keebio:Elite-C-castellated-24pin-holes
Connections:
- U1 pad 10: unconnected-(U1-7/PE6-Pad10) -> Net-(J3-Pin_4)
- U1 pad 11: unconnected-(U1-8/PB4-Pad11) -> Net-(J3-Pin_5)
- U1 pad 12: unconnected-(U1-9/PB5-Pad12) -> Net-(J3-Pin_6)
- U1 pad 13: Net-(J1-Pin_17) -> Net-(U1-10/PB6)
- U1 pad 14: Net-(J1-Pin_18) -> Net-(U1-16/PB2)
- U1 pad 15: Net-(J1-Pin_19) -> Net-(U1-14/PB3)
- U1 pad 16: Net-(J1-Pin_20) -> Net-(U1-15/PB1)
- U1 pad 17: Net-(J1-Pin_21) -> Net-(U1-A0/PF7)
- U1 pad 18: Net-(J1-Pin_22) -> Net-(U1-A1/PF6)
- U1 pad 19: Net-(J1-Pin_23) -> Net-(U1-A2/PF5)
- U1 pad 20: Net-(J1-Pin_24) -> Net-(U1-A3/PF4)
- U1 pad 21: +5V -> VCC
- U1 pad 24: unconnected-(U1-B0-Pad24) -> VBUS
- U1 pad 9: unconnected-(U1-6/PD7-Pad9) -> Net-(J3-Pin_3)
- U3 pad 16: +5V -> VBUS
- U3 pad 6: +5V -> VCC
- U4 pad 16: +5V -> VBUS
Routing:
- net Net-(J3-Pin_6): track 0.00 -> 75.8 mm, vias 0 -> 1
- net VBUS: track 0.00 -> 71.2 mm, vias 0 -> 4
- net Net-(J3-Pin_5): track 0.00 -> 69.7 mm, vias 0 -> 1
- net GND: track 68.9 -> 136.4 mm, vias 12 -> 20
- net Net-(J3-Pin_4): track 0.00 -> 61.1 mm, vias 0 -> 1
- net Net-(J3-Pin_3): track 0.00 -> 53.8 mm, vias 0 -> 1
- net +5V: track 52.5 -> 0.00 mm, vias 2 -> 0
- net VCC: track 0.00 -> 52.0 mm, vias 0 -> 2
- net Net-(J1-Pin_24): track 37.3 -> 6.51 mm
- net Net-(J1-Pin_23): track 31.2 -> 4.31 mm
- net Net-(U1-A3/PF4): track 0.00 -> 24.4 mm, vias 0 -> 2
- net Net-(J1-Pin_22): track 30.6 -> 6.49 mm
- net Net-(J1-Pin_20): track 28.5 -> 6.27 mm, vias 1 -> 0
- net Net-(U1-A2/PF5): track 0.00 -> 22.0 mm
- net Net-(J1-Pin_21): track 25.5 -> 4.02 mm
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