File: 24_wires_away.kicad_sch (KiCad schematic)
At the start: 4 parts, among them J1 Conn_01x24_Pin, U1 Elite-C, U3 74HCT138, U4 74HCT138

Commit message: more changes
Parts:
- added J3: Conn_01x06_Pin, Library:SolderWire-SMD-0.127sqmm_1x06_P3.7mm_D0.48mm_OD1mm, symbol Connector:Conn_01x06_Pin
- added U2: TXS0108EPW, Package_SO:TSSOP-20_4.4x6.5mm_P0.65mm, symbol Logic_LevelTranslator:TXS0108EPW
- U1: footprint Keebio:Elite-C-castellated-24pin -> Keebio:Elite-C-castellated-24pin-holes
Connections:
- net GND: now also J3.2 (Pin_2), U2.10 (OE), U2.11 (GND)
- net at U1.10 (7/PE6): now also J3.4 (Pin_4)
- net at U1.11 (8/PB4): now also J3.5 (Pin_5)
- net at U1.12 (9/PB5): now also J3.6 (Pin_6)
- net at U1.13 (10/PB6): now also U2.9 (A8); no longer J1.17 (Pin_17)
- net at U1.14 (16/PB2): now also U2.8 (A7); no longer J1.18 (Pin_18)
- net at U1.15 (14/PB3): now also U2.7 (A6); no longer J1.19 (Pin_19)
- net at U1.16 (15/PB1): now also U2.6 (A5); no longer J1.20 (Pin_20)
- net at U1.17 (A0/PF7): now also U2.5 (A4); no longer J1.21 (Pin_21)
- net at U1.18 (A1/PF6): now also U2.4 (A3); no longer J1.22 (Pin_22)
- net at U1.19 (A2/PF5): now also U2.3 (A2); no longer J1.23 (Pin_23)
- net at U1.20 (A3/PF4): now also U2.1 (A1); no longer J1.24 (Pin_24)
- net VBUS: now reaches U1.24 (B0)
- net VBUS: now also U3.16 (VCC), U4.16 (VCC), J3.1 (Pin_1), U2.19 (VCCB)
- net at U1.9 (6/PD7): now also J3.3 (Pin_3)
- net +5V renamed VCC
- net VCC: now also U2.2 (VCCA); no longer U3.16 (VCC), U4.16 (VCC)
- new net: J1.17 (Pin_17), U2.12 (B8)
- new net: J1.18 (Pin_18), U2.13 (B7)
- new net: J1.19 (Pin_19), U2.14 (B6)
- new net: J1.20 (Pin_20), U2.15 (B5)
- new net: J1.21 (Pin_21), U2.16 (B4)
- new net: J1.22 (Pin_22), U2.17 (B3)
- new net: J1.23 (Pin_23), U2.18 (B2)
- new net: J1.24 (Pin_24), U2.20 (B1)
- no-connect marks 0 -> 8
Other:
- moved on the sheet: J1, U1, U3, U4
