File: 24_wires_away.kicad_sch (KiCad schematic)
At the start: 6 parts, among them J1 Conn_01x24_Pin, J3 Conn_01x06_Pin, U1 Elite-C, U2 TXS0108EPW, U3 74HCT138, U4 74HCT138

Commit message: updated README.md
Parts:
- added C1, C2, C3: 100n, Capacitor_SMD:C_0603_1608Metric, symbol Device:C
- added RN1, RN2: 10k, Resistor_SMD:R_Array_Convex_4x0603, symbol Device:R_Pack04
- U2: value TXS0108EPW -> 74LVC245APW; symbol Logic_LevelTranslator:TXS0108EPW -> 74xx:74HC245
Connections:
- net GND: now also U2.1 (A->B), U2.19 (CE), C1.2, C2.2, C3.2; no longer U2.11 (GND)
- net VBUS: now also C2.1, C3.1, RN1.5 (R4.2), RN1.6 (R3.2), RN1.7 (R2.2), RN1.8 (R1.2), RN2.5 (R4.2), RN2.6 (R3.2), RN2.7 (R2.2), RN2.8 (R1.2); no longer U2.19 (VCCB)
- net VCC: now also U2.20 (VCC), C1.1; no longer U2.2 (VCCA)
- net at U1.20 (A3/PF4): now also U2.2 (A0); no longer U2.1 (A1)
- net COL7: now reaches U2.12 (B6)
- net COL7: now also J1.18 (Pin_18), RN2.3 (R3.1); no longer J1.17 (Pin_17)
- net COL6: now reaches U2.13 (B5)
- net COL6: now also J1.19 (Pin_19), RN2.2 (R2.1); no longer J1.18 (Pin_18)
- net COL5: now reaches U2.14 (B4)
- net COL5: now also J1.20 (Pin_20), RN2.1 (R1.1); no longer J1.19 (Pin_19)
- net COL4: now reaches U2.15 (B3)
- net COL4: now also J1.21 (Pin_21), RN1.4 (R4.1); no longer J1.20 (Pin_20)
- net COL3: now reaches U2.16 (B2)
- net COL3: now also J1.22 (Pin_22), RN1.3 (R3.1); no longer J1.21 (Pin_21)
- net COL2: now reaches U2.17 (B1)
- net COL2: now also J1.23 (Pin_23), RN1.2 (R2.1); no longer J1.22 (Pin_22)
- net COL1: now reaches U2.18 (B0)
- net COL1: now also J1.24 (Pin_24), RN1.1 (R1.1); no longer J1.23 (Pin_23)
- new net COL8: J1.17 (Pin_17), RN2.4 (R4.1), U2.11 (B7)
